File: Copy of Info2P1Intento3.brd (EAGLE design)
At the start: 68.6 x 53.3 mm, 137 parts

Commit message: Funcion verificacion terminada
Connections:
- removed net N$62 (its old number): U1.5V, U2.10, U2.16, U3.10, U3.16, U4.10, U4.16, U5.10, U5.16, U6.10, U6.16, U7.10, U7.16, U8.10, U8.16, U9.10, U9.16
- new net N$140: U1.12, U2.10
- new net N$142: U1.5V, U2.16, U3.10, U3.16, U4.10, U4.16, U5.10, U5.16, U6.10, U6.16, U7.10, U7.16, U8.10, U8.16, U9.10, U9.16

Commit message: Version final programa
Connections:
- removed net N$142: U1.5V, U2.16, U3.10, U3.16, U4.10, U4.16, U5.10, U5.16, U6.10, U6.16, U7.10, U7.16, U8.10, U8.16, U9.10, U9.16
- net N$140: now also U1.5V, U2.16, U3.10, U3.16, U4.10, U4.16, U5.10, U5.16, U6.10, U6.16, U7.10, U7.16, U8.10, U8.16, U9.10, U9.16; no longer U1.12
